Commit message: update code to test

File: src/carrierbot_description/urdf/mobile_base.xacro (robot description, xacro)
@@ -6,6 +6,8 @@
     <xacro:property name="base_width" value="0.5" />
     <xacro:property name="base_height" value="0.19" />
-    <xacro:property name="wheel_radius" value="0.0865" />
-    <xacro:property name="wheel_length" value="0.07" />
+    <!-- v1 (robot_fablab) wheel geometry -->
+    <xacro:property name="wheel_radius" value="0.1" />
+    <xacro:property name="wheel_length" value="0.05" />
+    <xacro:property name="wheel_separation" value="0.57" />
     <xacro:property name="upper_base_length" value="0.21" />
     <xacro:property name="upper_base_width" value="0.29" />
@@ -98,5 +100,5 @@
         <parent link="base_link" />
         <child link="right_wheel_link" />
-        <origin xyz="0 ${-(base_width + wheel_length) / 2.0} 0" rpy="0 0 0" />
+        <origin xyz="0 ${-wheel_separation / 2.0} 0" rpy="0 0 0" />
         <axis xyz="0 1 0" />
     </joint>
@@ -104,5 +106,5 @@
         <parent link="base_link" />
         <child link="left_wheel_link" />
-        <origin xyz="0 ${(base_width + wheel_length) / 2.0} 0" rpy="0 0 0" />
+        <origin xyz="0 ${wheel_separation / 2.0} 0" rpy="0 0 0" />
         <axis xyz="0 1 0" />
     </joint>

File: src/carrierbot_description/urdf/mobile_base_gazebo.xacro (robot description, xacro)
@@ -22,10 +22,10 @@
         <xacro:if value="$(arg is_ignition)">
             <plugin filename="ign_ros2_control-system" name="ign_ros2_control::IgnitionROS2ControlPlugin">
-                <parameters>$(find carrierbot_controller)/config/robot_controller.yaml</parameters>
+                <parameters>$(find carrierbot_controller)/config/controller.yaml</parameters>
             </plugin>
         </xacro:if>
         <xacro:unless value="$(arg is_ignition)">
             <plugin filename="gz_ros2_control-system" name="gz_ros2_control::GazeboSimROS2ControlPlugin">
-                <parameters>$(find carrierbot_controller)/config/robot_controller.yaml</parameters>
+                <parameters>$(find carrierbot_controller)/config/controller.yaml</parameters>
             </plugin>
         </xacro:unless>

File: src/carrierbot_description/urdf/my_robot.urdf.xacro (robot description, xacro)
@@ -3,4 +3,5 @@
   <xacro:arg name="is_ignition" default="false"/>
   <xacro:arg name="is_sim" default="false"/>
+  <xacro:arg name="drive_mode" default="1"/>
   <xacro:include filename="common_properties.xacro" />
   <xacro:include filename="mobile_base.xacro" />

File: src/carrierbot_description/urdf/ros2_control.xacro (robot description, xacro)
@@ -19,10 +19,13 @@
                 <param name="port">/dev/usbcan</param>
                 <param name="baudrate">2000000</param>
+                <!-- robot_fablab_ws hardware launch uses mode 1; poll 0x050 @ 20 Hz -->
+                <param name="drive_mode">$(arg drive_mode)</param>
+                <param name="poll_period">0.05</param>
             </hardware>
         </xacro:unless>
         <joint name="base_right_wheel_joint">
             <command_interface name="velocity">
-                <param name="min">-1.0</param>
-                <param name="max">1.0</param>
+                <param name="min">-15.0</param>
+                <param name="max">15.0</param>
             </command_interface>
             <state_interface name="position"/>
@@ -31,6 +34,6 @@
         <joint name="base_left_wheel_joint">
             <command_interface name="velocity">
-                <param name="min">-1.0</param>
-                <param name="max">1.0</param>
+                <param name="min">-15.0</param>
+                <param name="max">15.0</param>
             </command_interface>
             <state_interface name="position"/>

File: src/carrierbot_description/urdf/sensors.xacro (robot description, xacro)
@@ -37,42 +37,76 @@
         </collision>
     </link>
+    <!-- v1 static TF (from robot_fablab amcl_localization.launch), expressed in base_link:
+         footprint->laser: (-0.17, 0, 0.6, yaw=pi)
+         footprint->imu:   (-0.17, 0.06, 0.6)
+         base_link is wheel_radius above footprint -->
     <joint name="laser_joint" type="fixed">
         <parent link="base_link" />
         <child link="laser" />
-        <origin xyz="${-base_length / 4.0} 0 ${base_height + 0.026}" rpy="0 0 0" />
+        <origin xyz="-0.17 0 ${0.6 - wheel_radius}" rpy="0 0 ${pi}" />
     </joint>
     <joint name="imu_joint" type="fixed">
         <parent link="base_link" />
         <child link="imu" />
-        <origin xyz="${-base_length / 4.0} 0 ${(base_height + 0.026) / 2.0}" rpy="0 0 0" />
+        <origin xyz="-0.17 0.06 ${0.6 - wheel_radius}" rpy="0 0 0" />
     </joint>
-    <gazebo reference="laser">
-        <sensor name="laser" type="ray">
-            <pose> 0 0 0 0 0 0 </pose>
-            <visualize>true</visualize>
-            <update_rate>10.0</update_rate>
-            <ray>
-                <scan>
-                    <horizontal>
-                        <sample>720</sample>
+    <!-- Gazebo Sim sensor. ros_gz_bridge exposes /scan to ROS 2. -->
+    <xacro:if value="$(arg is_ignition)">
+        <gazebo reference="laser">
+            <sensor name="laser" type="gpu_lidar">
+                <pose>0 0 0 0 0 0</pose>
+                <topic>/scan</topic>
+                <visualize>true</visualize>
+                <update_rate>10.0</update_rate>
+                <ray>
+                    <scan>
+                        <horizontal>
+                            <samples>720</samples>
+                            <resolution>1</resolution>
+                            <min_angle>-3.14</min_angle>
+                            <max_angle>3.14</max_angle>
+                        </horizontal>
+                    </scan>
+                    <range>
+                        <min>0.5</min>
+                        <max>18.0</max>
+                        <resolution>0.01</resolution>
+                    </range>
+                </ray>
+                <always_on>true</always_on>
+            </sensor>
+        </gazebo>
+    </xacro:if>
+    <!-- Gazebo Classic fallback. -->
+    <xacro:unless value="$(arg is_ignition)">
+        <gazebo reference="laser">
+            <sensor name="laser" type="ray">
+                <pose>0 0 0 0 0 0</pose>
+                <visualize>true</visualize>
+                <update_rate>10.0</update_rate>
+                <ray>
+                    <scan>
+                        <horizontal>
+                            <sample>720</sample>
+                            <resolution>1</resolution>
+                            <min_angle>-3.14</min_angle>
+                            <max_angle>3.14</max_angle>
+                        </horizontal>
+                    </scan>
+                    <range>
+                        <min>0.5</min>
+                        <max>18.0</max>
                         <resolution>1</resolution>
-                        <min_angle>-3.14</min_angle>
-                        <max_angle>3.14</max_angle>
-                    </horizontal>
-                </scan>
-                <range>
-                    <min>0.5</min>
-                    <max>18.0</max>
-                    <resolution>1</resolution>
-                </range>
-            </ray>
-            <plugin name="laser_controller" filename="libgazebo_ros_ray_sensor.so">
-                <ros>
-                    <argument>~/out:=scan</argument>
-                </ros>
-                <output_type>sensor_msgs/LaserScan</output_type>
-                <frame_name>laser</frame_name>
-            </plugin>
-        </sensor>
-    </gazebo>
+                    </range>
+                </ray>
+                <plugin name="laser_controller" filename="libgazebo_ros_ray_sensor.so">
+                    <ros>
+                        <argument>~/out:=scan</argument>
+                    </ros>
+                    <output_type>sensor_msgs/LaserScan</output_type>
+                    <frame_name>laser</frame_name>
+                </plugin>
+            </sensor>
+        </gazebo>
+    </xacro:unless>
 </robot>
