Commit message: zed_usb2: set camera pitch fitted from B1 floor depth and limit depth to 3 m
Co-Authored-By: Claude Opus 5.5 <noreply@anthropic.com>

File: src/carrierbot_description/urdf/camera.xacro (robot description, xacro)
@@ -7,8 +7,9 @@
     <!-- Lens center height from the floor: robot top 1.57 m, camera just below it. -->
     <xacro:property name="camera_mount_height" value="1.54" />
-    <!-- Forward offset from base_link and pitch (negative = looking up) of the
-         camera on the slanted head; estimates, refine after measuring. -->
+    <!-- Forward offset from base_link (estimate) and pitch (negative = looking up)
+         of the camera on the slanted head.  Pitch ~12.6 deg up, fitted from the
+         floor in the B1 RTAB-Map depth images; refine after measuring. -->
     <xacro:property name="camera_mount_x" value="0.10" />
-    <xacro:property name="camera_mount_pitch" value="-0.35" />
+    <xacro:property name="camera_mount_pitch" value="-0.22" />
     <!-- Physical camera link -->
     <link name="camera_link">

Commit message: zed_usb2: camera is level, set measured pitch 0 in launch and URDF
Co-Authored-By: Claude Opus 5.5 <noreply@anthropic.com>

File: src/carrierbot_description/urdf/camera.xacro (robot description, xacro)
@@ -7,9 +7,9 @@
     <!-- Lens center height from the floor: robot top 1.57 m, camera just below it. -->
     <xacro:property name="camera_mount_height" value="1.54" />
-    <!-- Forward offset from base_link (estimate) and pitch (negative = looking up)
-         of the camera on the slanted head.  Pitch ~12.6 deg up, fitted from the
-         floor in the B1 RTAB-Map depth images; refine after measuring. -->
+    <!-- Forward offset from base_link (estimate) and pitch (negative = looking up).
+         Pitch measured level with a phone on top of the camera; the horizon in
+         the B1 camera images agrees. -->
     <xacro:property name="camera_mount_x" value="0.10" />
-    <xacro:property name="camera_mount_pitch" value="-0.22" />
+    <xacro:property name="camera_mount_pitch" value="0.0" />
     <!-- Physical camera link -->
     <link name="camera_link">
