Commit message: Add RGB-D camera support for Gazebo simulation

File: src/carrierbot_description/urdf/camera.xacro (robot description, xacro)
@@ -1,7 +1,9 @@
 <?xml version="1.0"?>
 <robot xmlns:xacro="http://www.ros.org/wiki/xacro">
+    <!-- Camera body dimensions -->
     <xacro:property name="camera_height" value="0.05" />
     <xacro:property name="camera_length" value="0.01" />
-    <xacro:property name="camera_width" value="0.1" />
+    <xacro:property name="camera_width" value="0.10" />
+    <!-- Physical camera link -->
     <link name="camera_link">
         <visual>
@@ -16,22 +18,96 @@
             </geometry>
         </collision>
-        <xacro:box_inertia m="0.1" l="${camera_length}" w="${camera_width}" h="${camera_height}"
-            xyz="0 0 0" rpy="0 0 0" />
+        <xacro:box_inertia
+            m="0.1"
+            l="${camera_length}"
+            w="${camera_width}"
+            h="${camera_height}"
+            xyz="0 0 0"
+            rpy="0 0 0" />
     </link>
+    <!-- Mount camera on robot -->
     <joint name="base_camera_joint" type="fixed">
         <parent link="base_link" />
         <child link="camera_link" />
-        <origin xyz="${(base_length + camera_length)/2.0 } 0 ${base_height/2.0}" rpy="0 0 0" />
+        <origin
+            xyz="${(base_length + camera_length) / 2.0} 0 ${base_height / 2.0}"
+            rpy="0 0 0" />
     </joint>
-    <gazebo reference="camera_link">
-        <material>Gazebo/Red</material>
-        <sensor name="camera_sensor" type="camera">
-            <pose>0 0 0 0 0 0</pose>
-            <visualize>true</visualize>
-            <update_rate>10.0</update_rate>
-            <plugin name="plugin_name" filename="libgazebo_ros_camera.so">
-                <frame_name>camera_link</frame_name>
-            </plugin>
-        </sensor>
-    </gazebo>
+    <!-- RGB optical frame -->
+    <link name="camera_rgb_optical_frame" />
+    <joint name="camera_rgb_optical_joint" type="fixed">
+        <parent link="camera_link" />
+        <child link="camera_rgb_optical_frame" />
+        <origin xyz="0 0 0" rpy="${-pi/2} 0 ${-pi/2}" />
+    </joint>
+    <!-- Depth optical frame -->
+    <link name="camera_depth_optical_frame" />
+    <joint name="camera_depth_optical_joint" type="fixed">
+        <parent link="camera_link" />
+        <child link="camera_depth_optical_frame" />
+        <origin xyz="0 0 0" rpy="${-pi/2} 0 ${-pi/2}" />
+    </joint>
+    <!-- Gazebo Classic RGB camera -->
+    <xacro:unless value="$(arg is_ignition)">
+        <gazebo reference="camera_link">
+            <material>Gazebo/Red</material>
+            <sensor name="rgb_camera" type="camera">
+                <always_on>true</always_on>
+                <visualize>true</visualize>
+                <update_rate>15.0</update_rate>
+                <camera name="rgb_camera">
+                    <horizontal_fov>1.047</horizontal_fov>
+                    <image>
+                        <width>640</width>
+                        <height>480</height>
+                        <format>R8G8B8</format>
+                    </image>
+                    <clip>
+                        <near>0.1</near>
+                        <far>20.0</far>
+                    </clip>
+                </camera>
+                <plugin
+                    name="rgb_camera_controller"
+                    filename="libgazebo_ros_camera.so">
+                    <ros>
+                        <remapping>~/image_raw:=/rgb/image_raw</remapping>
+                        <remapping>~/camera_info:=/rgb/camera_info</remapping>
+                    </ros>
+                    <camera_name>rgb</camera_name>
+                    <frame_name>camera_rgb_optical_frame</frame_name>
+                </plugin>
+            </sensor>
+            <!-- Depth camera -->
+            <sensor name="depth_camera" type="depth">
+                <always_on>true</always_on>
+                <visualize>true</visualize>
+                <update_rate>15.0</update_rate>
+                <camera name="depth_camera">
+                    <horizontal_fov>1.047</horizontal_fov>
+                    <image>
+                        <width>640</width>
+                        <height>480</height>
+                        <format>R8G8B8</format>
+                    </image>
+                    <clip>
+                        <near>0.1</near>
+                        <far>20.0</far>
+                    </clip>
+                </camera>
+                <plugin
+                    name="depth_camera_controller"
+                    filename="libgazebo_ros_camera.so">
+                    <ros>
+                        <remapping>~/image_depth:=/depth/image_raw</remapping>
+                        <remapping>~/camera_info_depth:=/depth/camera_info</remapping>
+                    </ros>
+                    <camera_name>depth</camera_name>
+                    <frame_name>camera_depth_optical_frame</frame_name>
+                    <min_depth>0.1</min_depth>
+                    <max_depth>20.0</max_depth>
+                </plugin>
+            </sensor>
+        </gazebo>
+    </xacro:unless>
 </robot>

File: src/carrierbot_description/urdf/mobile_base_gazebo.xacro (robot description, xacro)
@@ -27,5 +27,5 @@
         <xacro:unless value="$(arg is_ignition)">
             <plugin filename="libgazebo_ros2_control.so" name="gazebo_ros2_control">
-                <parameters>$(find carrierbot_controller)/config/controller.yaml</parameters>
+                <parameters>$(find carrierbot_controller)/config/controller_sim.yaml</parameters>
             </plugin>
         </xacro:unless>

File: src/carrierbot_description/urdf/my_robot.urdf.xacro (robot description, xacro)
@@ -9,5 +9,5 @@
   <xacro:include filename="mobile_base_gazebo.xacro" />
   <xacro:include filename="ros2_control.xacro" />
-  <!-- <xacro:include filename="camera.xacro" /> -->
+  <xacro:include filename="camera.xacro" />
   <xacro:include filename="sensors.xacro"/>
 </robot>

Commit message: fix run simulation 2d map

File: src/carrierbot_description/urdf/camera.xacro (robot description, xacro)
@@ -5,4 +5,6 @@
     <xacro:property name="camera_length" value="0.01" />
     <xacro:property name="camera_width" value="0.10" />
+    <!-- Measured from base_footprint; refine after measuring the physical mount. -->
+    <xacro:property name="camera_mount_height" value="1.10" />
     <!-- Physical camera link -->
     <link name="camera_link">
@@ -26,10 +28,10 @@
             rpy="0 0 0" />
     </link>
-    <!-- Mount camera on robot -->
+    <!-- Mount the camera above the front display, facing forward. -->
     <joint name="base_camera_joint" type="fixed">
         <parent link="base_link" />
         <child link="camera_link" />
         <origin
-            xyz="${(base_length + camera_length) / 2.0} 0 ${base_height / 2.0}"
+            xyz="${(base_length + camera_length) / 2.0} 0 ${camera_mount_height - wheel_radius}"
             rpy="0 0 0" />
     </joint>
@@ -52,9 +54,9 @@
         <gazebo reference="camera_link">
             <material>Gazebo/Red</material>
-            <sensor name="rgb_camera" type="camera">
+            <sensor name="rgbd_camera" type="depth">
                 <always_on>true</always_on>
-                <visualize>true</visualize>
+                <visualize>false</visualize>
                 <update_rate>15.0</update_rate>
-                <camera name="rgb_camera">
+                <camera name="rgbd_camera">
                     <horizontal_fov>1.047</horizontal_fov>
                     <image>
@@ -69,40 +71,14 @@
                 </camera>
                 <plugin
-                    name="rgb_camera_controller"
+                    name="rgbd_camera_controller"
                     filename="libgazebo_ros_camera.so">
                     <ros>
                         <remapping>~/image_raw:=/rgb/image_raw</remapping>
                         <remapping>~/camera_info:=/rgb/camera_info</remapping>
-                    </ros>
-                    <camera_name>rgb</camera_name>
-                    <frame_name>camera_rgb_optical_frame</frame_name>
-                </plugin>
-            </sensor>
-            <!-- Depth camera -->
-            <sensor name="depth_camera" type="depth">
-                <always_on>true</always_on>
-                <visualize>true</visualize>
-                <update_rate>15.0</update_rate>
-                <camera name="depth_camera">
-                    <horizontal_fov>1.047</horizontal_fov>
-                    <image>
-                        <width>640</width>
-                        <height>480</height>
-                        <format>R8G8B8</format>
-                    </image>
-                    <clip>
-                        <near>0.1</near>
-                        <far>20.0</far>
-                    </clip>
-                </camera>
-                <plugin
-                    name="depth_camera_controller"
-                    filename="libgazebo_ros_camera.so">
-                    <ros>
                         <remapping>~/image_depth:=/depth/image_raw</remapping>
                         <remapping>~/camera_info_depth:=/depth/camera_info</remapping>
                     </ros>
-                    <camera_name>depth</camera_name>
-                    <frame_name>camera_depth_optical_frame</frame_name>
+                    <camera_name>rgbd</camera_name>
+                    <frame_name>camera_rgb_optical_frame</frame_name>
                     <min_depth>0.1</min_depth>
                     <max_depth>20.0</max_depth>

File: src/carrierbot_description/urdf/sensors.xacro (robot description, xacro)
@@ -51,4 +51,21 @@
         <origin xyz="-0.17 0.06 ${0.6 - wheel_radius}" rpy="0 0 0" />
     </joint>
+    <!-- Gazebo Classic IMU. Publishes sensor_msgs/Imu on /imu/data. -->
+    <xacro:unless value="$(arg is_ignition)">
+        <gazebo reference="imu">
+            <sensor name="imu_sensor" type="imu">
+                <always_on>true</always_on>
+                <update_rate>100.0</update_rate>
+                <visualize>false</visualize>
+                <plugin name="imu_plugin" filename="libgazebo_ros_imu_sensor.so">
+                    <ros>
+                        <remapping>~/out:=imu/data</remapping>
+                    </ros>
+                    <frame_name>imu</frame_name>
+                    <initial_orientation_as_reference>false</initial_orientation_as_reference>
+                </plugin>
+            </sensor>
+        </gazebo>
+    </xacro:unless>
     <!-- Gazebo Sim sensor. ros_gz_bridge exposes /scan to ROS 2. -->
     <xacro:if value="$(arg is_ignition)">

Commit message: set measured ZED 2 mount height and estimated pitch in launch and URDF

File: src/carrierbot_description/urdf/camera.xacro (robot description, xacro)
@@ -5,6 +5,10 @@
     <xacro:property name="camera_length" value="0.01" />
     <xacro:property name="camera_width" value="0.10" />
-    <!-- Measured from base_footprint; refine after measuring the physical mount. -->
-    <xacro:property name="camera_mount_height" value="1.10" />
+    <!-- Lens center height from the floor: robot top 1.57 m, camera just below it. -->
+    <xacro:property name="camera_mount_height" value="1.54" />
+    <!-- Forward offset from base_link and pitch (negative = looking up) of the
+         camera on the slanted head; estimates, refine after measuring. -->
+    <xacro:property name="camera_mount_x" value="0.10" />
+    <xacro:property name="camera_mount_pitch" value="-0.35" />
     <!-- Physical camera link -->
     <link name="camera_link">
@@ -33,6 +37,6 @@
         <child link="camera_link" />
         <origin
-            xyz="${(base_length + camera_length) / 2.0} 0 ${camera_mount_height - wheel_radius}"
-            rpy="0 0 0" />
+            xyz="${camera_mount_x} 0 ${camera_mount_height - wheel_radius}"
+            rpy="0 ${camera_mount_pitch} 0" />
     </joint>
     <!-- RGB optical frame -->

Commit message: add code sim

File: src/carrierbot_description/urdf/camera.xacro (robot description, xacro)
@@ -12,4 +12,13 @@
     <xacro:property name="camera_mount_x" value="0.10" />
     <xacro:property name="camera_mount_pitch" value="0.0" />
+    <!-- Simulated RGB-D matched to the real ZED 2 pipeline (zed_usb2_rgbd.py):
+         VGA 672x376, depth limited to 0.3-3.0 m (max_depth in zed_usb2_rgbd.launch.py).
+         HFOV = 2*atan(336/fx). fx ~ 264 px is the usual ZED 2 VGA value; confirm with the
+         "rectified fx" line that zed_usb2_rgbd prints at startup on the robot. -->
+    <xacro:property name="camera_hfov" value="1.81" />
+    <xacro:property name="camera_image_width" value="672" />
+    <xacro:property name="camera_image_height" value="376" />
+    <xacro:property name="camera_min_depth" value="0.3" />
+    <xacro:property name="camera_max_depth" value="3.0" />
     <!-- Physical camera link -->
     <link name="camera_link">
@@ -64,8 +73,8 @@
                 <update_rate>15.0</update_rate>
                 <camera name="rgbd_camera">
-                    <horizontal_fov>1.047</horizontal_fov>
+                    <horizontal_fov>${camera_hfov}</horizontal_fov>
                     <image>
-                        <width>640</width>
-                        <height>480</height>
+                        <width>${camera_image_width}</width>
+                        <height>${camera_image_height}</height>
                         <format>R8G8B8</format>
                     </image>
@@ -88,6 +97,6 @@
                     <camera_name>rgbd</camera_name>
                     <frame_name>camera_rgb_optical_frame</frame_name>
-                    <min_depth>0.1</min_depth>
-                    <max_depth>20.0</max_depth>
+                    <min_depth>${camera_min_depth}</min_depth>
+                    <max_depth>${camera_max_depth}</max_depth>
                 </plugin>
             </sensor>

File: src/carrierbot_description/urdf/sensors.xacro (robot description, xacro)
@@ -3,4 +3,12 @@
     <xacro:property name="lidar_height" value="0.037" />
     <xacro:property name="lidar_radius" value="0.0345" />
+    <!-- Simulated scan matched to the real RPLidar S2 (real_robot.launch.py):
+         DenseBoost at 10 Hz gives 3200 points per turn (0.1125 deg).
+         Range 0.5-12 m is what laser_filter keeps on the real robot.
+         Noise 0.01 m std is about the S2 datasheet accuracy (+-30 mm). -->
+    <xacro:property name="lidar_samples" value="3200" />
+    <xacro:property name="lidar_min_range" value="0.5" />
+    <xacro:property name="lidar_max_range" value="12.0" />
+    <xacro:property name="lidar_noise_std" value="0.01" />
     <!-- Include lidar -->
     <link name="laser">
@@ -79,5 +87,5 @@
                     <scan>
                         <horizontal>
-                            <samples>720</samples>
+                            <samples>${lidar_samples}</samples>
                             <resolution>1</resolution>
                             <min_angle>-3.14</min_angle>
@@ -86,6 +94,6 @@
                     </scan>
                     <range>
-                        <min>0.5</min>
-                        <max>18.0</max>
+                        <min>${lidar_min_range}</min>
+                        <max>${lidar_max_range}</max>
                         <resolution>0.01</resolution>
                     </range>
@@ -105,5 +113,5 @@
                     <scan>
                         <horizontal>
-                        <samples>720</samples>
+                        <samples>${lidar_samples}</samples>
                             <resolution>1</resolution>
                             <min_angle>-3.14</min_angle>
@@ -112,8 +120,13 @@
                     </scan>
                     <range>
-                        <min>0.5</min>
-                        <max>18.0</max>
+                        <min>${lidar_min_range}</min>
+                        <max>${lidar_max_range}</max>
                         <resolution>1</resolution>
                     </range>
+                    <noise>
+                        <type>gaussian</type>
+                        <mean>0.0</mean>
+                        <stddev>${lidar_noise_std}</stddev>
+                    </noise>
                 </ray>
                 <plugin name="laser_controller" filename="libgazebo_ros_ray_sensor.so">
